File: hardware/hivis2smd.kicad_sch (KiCad schematic)
At the start: 15 parts, among them J1 BME_688_Module, J2 INMP_441, J3 OLED Display, J4 J5019_Module, J5 JST_PH2.0_BATT, SW1 SW_Push

Commit message: Add SMD variant: schematic, Gerbers, BOM, and production files
Updated KiCad project files with SMD components. New files:
- hivis2smd.kicad_sch — SMD schematic
- gerbers/smd/ — SMD Gerber set + zip
- gerbers/hivistht.zip — THT Gerber zip
- production/ — BOM, positions, netlist, and fabrication zip
- hivis2smdBOM.csv, top/bottom position CSVs

Co-Authored-By: Claude Sonnet 4.6 <noreply@anthropic.com>
Parts:
- C1, C2: footprint Capacitor_SMD:C_0402_1005Metric -> Capacitor_THT:C_Disc_D5.0mm_W2.5mm_P5.00mm
- R1, R2, R3, R4, R5: footprint Resistor_SMD:R_0402_1005Metric -> Resistor_THT:R_Axial_DIN0204_L3.6mm_D1.6mm_P7.62mm_Horizontal
- U1: footprint ESP32_Footprints:ESP32_30pin -> ESP32_30pin
Changed lines of the file:
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@@
 			)
 		)
-		(property "Footprint" "Resistor_SMD:R_0402_1005Metric"
+		(property "Footprint" "Resistor_THT:R_Axial_DIN0204_L3.6mm_D1.6mm_P7.62mm_Horizontal"
 			(at 162.052 68.58 90)
 			(effects
@@
 			)
 		)
-		(property "Footprint" "Resistor_SMD:R_0402_1005Metric"
+		(property "Footprint" "Resistor_THT:R_Axial_DIN0204_L3.6mm_D1.6mm_P7.62mm_Horizontal"
 			(at 170.942 68.58 90)
 			(effects
@@
 			)
 		)
-		(property "Footprint" "Resistor_SMD:R_0402_1005Metric"
+		(property "Footprint" "Resistor_THT:R_Axial_DIN0204_L3.6mm_D1.6mm_P7.62mm_Horizontal"
 			(at 71.882 88.9 90)
 			(effects
@@
 			)
 		)
-		(property "Footprint" "Capacitor_SMD:C_0402_1005Metric"
+		(property "Footprint" "Capacitor_THT:C_Disc_D5.0mm_W2.5mm_P5.00mm"
 			(at 204.1652 44.45 0)
 			(effects
@@
 			)
 		)
-		(property "Footprint" "ESP32_Footprints:ESP32_30pin"
+		(property "Footprint" "ESP32_30pin"
 			(at 132.08 56.515 0)
 			(effects
@@
 			)
 		)
-		(property "Footprint" "Resistor_SMD:R_0402_1005Metric"
+		(property "Footprint" "Resistor_THT:R_Axial_DIN0204_L3.6mm_D1.6mm_P7.62mm_Horizontal"
 			(at 85.852 71.12 90)
 			(effects
@@
 			)
 		)
-		(property "Footprint" "Capacitor_SMD:C_0402_1005Metric"
+		(property "Footprint" "Capacitor_THT:C_Disc_D5.0mm_W2.5mm_P5.00mm"
 			(at 169.8752 38.1 0)
 			(effects
@@
 			)
 		)
-		(property "Footprint" "Resistor_SMD:R_0402_1005Metric"
+		(property "Footprint" "Resistor_THT:R_Axial_DIN0204_L3.6mm_D1.6mm_P7.62mm_Horizontal"
 			(at 85.852 63.5 90)
 			(effects
